Commit message: about to try adding kinematic controller for gazebo

File: asc_description/urdf/asc_description.urdf (robot description, URDF)
Before this commit: robot asc_description, 7 links, 6 joints
Links:
- added link front_steer_link; visual mesh filename=package://asc_description/meshes/right_rear_wheel.STL
- added link rear_steer_link; visual mesh filename=package://asc_description/meshes/right_rear_wheel.STL
Joints:
- removed joint left_rear_wheel
- added joint front_steer_joint: type fixed, parent base_link, child front_steer_link, origin xyz=1.186 0 -0.409 rpy=0 0 0
- added joint left_rear_wheel_joint: type continuous, parent base_link, child left_rear_wheel, origin xyz=-1.3237 0.70906 -0.41261 rpy=3.1416 0.12841 3.1416, axis 0 1 0
- added joint rear_wheel_joint: type fixed, parent base_link, child rear_steer_link, origin xyz=-1.3237 0 -0.41261 rpy=0 0 0
- joint left_front_steering_joint: origin xyz=0.9825 0.63618 0.047063 rpy=0.13336 -0.28845 0.0036248 -> xyz=0.9825 0.63618 0.047063 rpy=0.13546 -0.28749 0.0037802

Commit message: need to add xacro file

File: asc_description/urdf/asc_description.urdf (robot description, URDF)
Before this commit: robot asc_description, 9 links, 8 joints
Links:
- removed link front_steer_link
- removed link rear_steer_link
Joints:
- removed joint front_steer_joint
- removed joint rear_wheel_joint
- removed joint right_rear_wheel
- added joint right_rear_wheel_joint: type continuous, parent base_link, child right_rear_wheel, origin xyz=-1.3237 -0.70606 -0.41261 rpy=0 0.12841 3.1416, axis 0 1 0

Commit message: major update, several added transmissions as well as PID config

File: asc_description/urdf/asc_description.urdf (robot description, URDF)
Before this commit: robot asc_description, 7 links, 6 joints
Links:
- link base_link: geometry visual mesh filename=package://asc_description/meshes/base_link.STL
- link left_front_wheel_link: geometry collision cylinder length=0.05 radius=0.3; visual cylinder length=0.05 radius=0.3
- link left_rear_wheel: geometry collision cylinder length=0.05 radius=0.3; visual cylinder length=0.05 radius=0.3
- link right_front_wheel_link: geometry collision cylinder length=0.05 radius=0.3; visual cylinder length=0.05 radius=0.3
- link right_rear_wheel: geometry collision cylinder length=0.05 radius=0.3; visual cylinder length=0.05 radius=0.3
Joints:
- removed joint right_front_wheel_link
- added joint right_front_wheel_joint: type continuous, parent right_front_steering_link, child right_front_wheel_link, origin xyz=0.065291 -0.059582 -0.50741 rpy=1.8455 1.0552 0.23683, axis 0 0 1

Commit message: controllers work, trying move_base next

File: asc_description/urdf/asc_description.urdf (robot description, URDF)
Before this commit: robot asc, 7 links, 6 joints
Links:
- added link frame_link, mass 54.6845003989778; visual mesh filename=package://asc_description/meshes/base_link.STL
- added link left_rear_steer, mass 1
- added link right_rear_steer, mass 1
- link base_link: mass 54.6845003989778 -> None; geometry 
Joints:
- added joint base_link_to_frame: type fixed, parent base_link, child frame_link, origin xyz=0 0 1 rpy=0 0 0, axis 0 0 1
- added joint left_rear_steering_joint: type revolute, parent frame_link, child left_rear_steer, origin xyz=-1.3237 0.70906 -0.41261 rpy=0 0 0, axis 0 0 1, limit lower=0 upper=0 effort=0 velocity=0
- added joint right_rear_steering_joint: type revolute, parent frame_link, child right_rear_steer, origin xyz=-1.3237 -0.70606 -0.41261 rpy=0 0 0, axis 0 0 1, limit lower=0 upper=0 effort=0 velocity=0
- joint left_front_steering_joint: limit lower=-1.57 upper=1.57 effort=0 velocity=0 -> lower=-0.8 upper=0.9 effort=100 velocity=100; parent base_link -> frame_link
- joint left_rear_wheel_joint: origin xyz=-1.3237 0.70906 -0.41261 rpy=3.1416 0.12841 3.1416 -> xyz=0 0 0 rpy=0 0 0; parent base_link -> left_rear_steer
- joint right_front_steering_joint: limit lower=-1.57 upper=1.57 effort=0 velocity=0 -> lower=-0.8 upper=0.8 effort=100 velocity=100; parent base_link -> frame_link
- joint right_rear_wheel_joint: origin xyz=-1.3237 -0.70606 -0.41261 rpy=0 0.12841 3.1416 -> xyz=0 0 0 rpy=0 0 0; parent base_link -> right_rear_steer
