Commit message: moved to xacro

File: asc_description/urdf/asc.urdf.xacro (robot description, xacro)
@@ -1,3 +1,358 @@
 <?xml version="1.0"?>
-<robot name="robot" xmlns:xacro="http://www.ros.org/wiki/xacro">
+<robot xmlns:xacro="http://www.ros.org/wiki/xacro" name="robot">
+  <gazebo>
+    <plugin name="gazebo_ros_control" filename="libgazebo_ros_control.so">
+      <robotNamespace>/asc</robotNamespace>
+      <!--<robotParam>/robot_description</robotParam> -->
+      <robotSimType>gazebo_ros_control/DefaultRobotHWSim</robotSimType>
+    </plugin>
+  </gazebo>
+  <link name="base_link"/>
+  <joint name="base_link_to_frame" type="fixed">
+    <origin xyz="0 0 1" rpy="0 0 0"/>
+    <parent link="base_link"/>
+    <child link="frame_link"/>
+    <axis xyz="0 0 1"/>
+  </joint>
+  <link name="frame_link">
+    <inertial>
+      <origin xyz="-0.191135074026536 0.00147037627768998 -0.144166350352701" rpy="0 0 0"/>
+      <mass value="54.6845003989778"/>
+      <inertia ixx="0.830289508168532" ixy="-7.44170925374484E-07" ixz="-0.168031775231281" iyy="1.89493024064907" iyz="3.6787232173372E-07" izz="1.80540947379668"/>
+    </inertial>
+    <visual>
+      <origin xyz="0 0 0" rpy="0 0 0"/>
+      <geometry>
+        <mesh filename="package://asc_description/meshes/base_link.STL"/>
+      </geometry>
+      <material name="">
+        <color rgba="0.866666666666667 0.866666666666667 0.890196078431372 1"/>
+      </material>
+    </visual>
+    <!--
+    <collision>
+      <origin xyz="0 0 0" rpy="0 0 0"/>
+      <geometry>
+        <mesh filename="package://asc_description/meshes/base_link.STL"/>
+      </geometry>
+    </collision> -->
+  </link>
+  <link name="left_front_steering_link">
+    <inertial>
+      <origin xyz="-0.0439194980427094 -0.0123148656628935 -0.29574701698731" rpy="0 0 0"/>
+      <mass value="5.71439015182903"/>
+      <inertia ixx="0.138973038944984" ixy="0.00240438901312515" ixz="0.0320681563279578" iyy="0.160053837434921" iyz="-0.0109556260035955" izz="0.028546837728721"/>
+    </inertial>
+    <visual>
+      <origin xyz="0 0 0" rpy="0 0 0"/>
+      <geometry>
+        <mesh filename="package://asc_description/meshes/left_front_steering_link.STL"/>
+      </geometry>
+      <material name="">
+        <color rgba="0.792156862745098 0.819607843137255 0.933333333333333 1"/>
+      </material>
+    </visual>
+    <collision>
+      <origin xyz="0 0 0" rpy="0 0 0"/>
+      <geometry>
+        <mesh filename="package://asc_description/meshes/left_front_steering_link.STL"/>
+      </geometry>
+    </collision>
+  </link>
+  <joint name="left_front_steering_joint" type="revolute">
+    <origin xyz="0.9825 0.63618 0.047063" rpy="0.13546 -0.28749 0.0037802"/>
+    <parent link="frame_link"/>
+    <child link="left_front_steering_link"/>
+    <axis xyz="0 0 1"/>
+    <limit lower="-0.8" upper="0.9" effort="100" velocity="100"/>
+  </joint>
+  <link name="left_front_wheel_link">
+    <inertial>
+      <origin xyz="-2.26485497023532E-14 4.10782519111308E-14 0.00509989314954018" rpy="0 0 0"/>
+      <mass value="3.6905479088754"/>
+      <inertia ixx="0.117114266308146" ixy="-6.93889390390723E-18" ixz="1.02756637900478E-17" iyy="0.117114266308146" iyz="-3.62378420062206E-17" izz="0.227951064044091"/>
+    </inertial>
+    <visual>
+      <origin xyz="0 0 0" rpy="0 0 0"/>
+      <geometry>
+        <cylinder length="0.05" radius="0.3"/>
+      </geometry>
+    </visual>
+    <collision>
+      <origin xyz="0 0 0" rpy="0 0 0"/>
+      <geometry>
+        <cylinder length="0.05" radius="0.3"/>
+      </geometry>
+    </collision>
+  </link>
+  <joint name="left_front_wheel_joint" type="continuous">
+    <origin xyz="0.065693 0.065054 -0.50813" rpy="-1.8471 1.0585 -0.24589"/>
+    <parent link="left_front_steering_link"/>
+    <child link="left_front_wheel_link"/>
+    <axis xyz="0 0 1"/>
+  </joint>
+  <link name="right_front_steering_link">
+    <inertial>
+      <origin xyz="-0.0465182122250822 0.0145095544427134 -0.290619703564971" rpy="0 0 0"/>
+      <mass value="5.57746367002881"/>
+      <inertia ixx="0.138857493635095" ixy="-0.0022557465179349" ixz="0.032139397456901" iyy="0.160001336296301" iyz="0.0107272499121531" izz="0.0284811002523076"/>
+    </inertial>
+    <visual>
+      <origin xyz="0 0 0" rpy="0 0 0"/>
+      <geometry>
+        <mesh filename="package://asc_description/meshes/right_front_steering_link.STL"/>
+      </geometry>
+      <material name="">
+        <color rgba="0.792156862745098 0.819607843137255 0.933333333333333 1"/>
+      </material>
+    </visual>
+    <collision>
+      <origin xyz="0 0 0" rpy="0 0 0"/>
+      <geometry>
+        <mesh filename="package://asc_description/meshes/right_front_steering_link.STL"/>
+      </geometry>
+    </collision>
+  </link>
+  <joint name="right_front_steering_joint" type="revolute">
+    <origin xyz="0.9825 -0.63318 0.047063" rpy="-0.13546 -0.28749 0.0037802"/>
+    <parent link="frame_link"/>
+    <child link="right_front_steering_link"/>
+    <axis xyz="0 0 1"/>
+    <limit lower="-0.8" upper="0.8" effort="100" velocity="100"/>
+  </joint>
+  <link name="right_front_wheel_link">
+    <inertial>
+      <origin xyz="-1.02140518265514E-14 6.85007606193722E-14 0.00509989314946457" rpy="0 0 0"/>
+      <mass value="3.69054790887537"/>
+      <inertia ixx="0.117114266308143" ixy="1.38777878078145E-17" ixz="2.37549730750149E-18" iyy="0.117114266308143" iyz="3.40770700491441E-17" izz="0.22795106404409"/>
+    </inertial>
+    <visual>
+      <origin xyz="0 0 0" rpy="0 0 0"/>
+      <geometry>
+        <cylinder length="0.05" radius="0.3"/>
+      </geometry>
+    </visual>
+    <collision>
+      <origin xyz="0 0 0" rpy="0 0 0"/>
+      <geometry>
+        <cylinder length="0.05" radius="0.3"/>
+      </geometry>
+    </collision>
+  </link>
+  <joint name="right_front_wheel_joint" type="continuous">
+    <origin xyz="0.065291 -0.059582 -0.50741" rpy="1.8455 1.0552 0.23683"/>
+    <parent link="right_front_steering_link"/>
+    <child link="right_front_wheel_link"/>
+    <axis xyz="0 0 1"/>
+  </joint>
+  <!-- add fake rear steering joint-->
+  <link name="left_rear_steer">
+    <inertial>
+      <origin xyz="0 0 0" rpy="0 0 0"/>
+      <mass value="1"/>
+      <inertia ixx="1.0" ixy="0.0" ixz="0.0" iyy="1.0" iyz="0.0" izz="1.0"/>
+    </inertial>
+  </link>
+  <joint name="left_rear_steering_joint" type="revolute">
+    <origin xyz="-1.3237 0.70906 -0.41261" rpy="0 0 0"/>
+    <parent link="frame_link"/>
+    <child link="left_rear_steer"/>
+    <axis xyz="0 0 1"/>
+    <limit lower="0" upper="0" effort="0" velocity="0"/>
+  </joint>
+  <link name="left_rear_wheel">
+    <inertial>
+      <origin xyz="8.43769498715119E-15 0.0589722640664191 -5.01820807130571E-14" rpy="0 0 0"/>
+      <mass value="3.68939811577995"/>
+      <inertia ixx="0.117113236563891" ixy="-4.42261767048626E-17" ixz="-6.93889390390723E-18" iyy="0.227950884881602" iyz="-3.11187820789416E-16" izz="0.117113236563891"/>
+    </inertial>
+    <visual>
+      <origin xyz="0 0 0" rpy="1.57 0 0"/>
+      <geometry>
+        <cylinder length="0.05" radius="0.3"/>
+      </geometry>
+    </visual>
+    <collision>
+      <origin xyz="0 0 0" rpy="1.57 0 0"/>
+      <geometry>
+        <cylinder length="0.05" radius="0.3"/>
+      </geometry>
+    </collision>
+  </link>
+  <joint name="left_rear_wheel_joint" type="continuous">
+    <origin xyz="0 0 0" rpy="0 0 0"/>
+    <parent link="left_rear_steer"/>
+    <child link="left_rear_wheel"/>
+    <axis xyz="0 1 0"/>
+  </joint>
+  <!-- add fake rear steering joint-->
+  <link name="right_rear_steer">
+    <inertial>
+      <origin xyz="0 0 0" rpy="0 0 0"/>
+      <mass value="1"/>
+      <inertia ixx="1.0" ixy="0.0" ixz="0.0" iyy="1.0" iyz="0.0" izz="1.0"/>
+    </inertial>
+  </link>
+  <joint name="right_rear_steering_joint" type="revolute">
+    <origin xyz="-1.3237 -0.70606 -0.41261" rpy="0 0 0"/>
+    <parent link="frame_link"/>
+    <child link="right_rear_steer"/>
+    <axis xyz="0 0 1"/>
+    <limit lower="0" upper="0" effort="0" velocity="0"/>
+  </joint>
+  <link name="right_rear_wheel">
+    <inertial>
+      <origin xyz="7.99360577730113E-15 0.0589722640664192 4.2410519540681E-14" rpy="0 0 0"/>
+      <mass value="3.68939811577991"/>
+      <inertia ixx="0.117113236563893" ixy="-4.66966016159301E-17" ixz="4.33680868994202E-18" iyy="0.2279508848816" iyz="3.34438350256477E-16" izz="0.117113236563893"/>
+    </inertial>
+    <visual>
+      <origin xyz="0 0 0" rpy="1.57 0 0"/>
+      <geometry>
+        <cylinder length="0.05" radius="0.3"/>
+      </geometry>
+    </visual>
+    <collision>
+      <origin xyz="0 0 0" rpy="1.57 0 0"/>
+      <geometry>
+        <cylinder length="0.05" radius="0.3"/>
+      </geometry>
+    </collision>
+  </link>
+  <joint name="right_rear_wheel_joint" type="continuous">
+    <origin xyz="0 0 0" rpy="0 0 0"/>
+    <parent link="right_rear_steer"/>
+    <child link="right_rear_wheel"/>
+    <axis xyz="0 1 0"/>
+  </joint>
+  <transmission name="tran1">
+    <type>transmission_interface/SimpleTransmission</type>
+    <joint name="left_rear_wheel_joint">
+      <hardwareInterface>hardware_interface/VelocityJointInterface</hardwareInterface>
+    </joint>
+    <actuator name="motor1">
+      <hardwareInterface>hardware_interface/VelocityJointInterface</hardwareInterface>
+      <mechanicalReduction>1</mechanicalReduction>
+    </actuator>
+  </transmission>
+  <transmission name="tran2">
+    <type>transmission_interface/SimpleTransmission</type>
+    <joint name="right_rear_wheel_joint">
+      <hardwareInterface>hardware_interface/VelocityJointInterface</hardwareInterface>
+    </joint>
+    <actuator name="motor2">
+      <hardwareInterface>hardware_interface/VelocityJointInterface</hardwareInterface>
+      <mechanicalReduction>1</mechanicalReduction>
+    </actuator>
+  </transmission>
+  <!-- Transmissions for steering joints-->
+  <transmission name="tran3">
+    <type>transmission_interface/SimpleTransmission</type>
+    <joint name="left_front_steering_joint">
+      <hardwareInterface>hardware_interface/PositionJointInterface</hardwareInterface>
+    </joint>
+    <actuator name="motor3">
+      <hardwareInterface>hardware_interface/PositionJointInterface</hardwareInterface>
+      <mechanicalReduction>1</mechanicalReduction>
+    </actuator>
+  </transmission>
+  <transmission name="tran4">
+    <type>transmission_interface/SimpleTransmission</type>
+    <joint name="right_front_steering_joint">
+      <hardwareInterface>hardware_interface/PositionJointInterface</hardwareInterface>
+    </joint>
+    <actuator name="motor4">
+      <hardwareInterface>hardware_interface/PositionJointInterface</hardwareInterface>
+      <mechanicalReduction>1</mechanicalReduction>
+    </actuator>
+  </transmission>
+  <!-- Transmissions for fake steering joints-->
+  <transmission name="tran5">
+    <type>transmission_interface/SimpleTransmission</type>
+    <joint name="left_rear_steering_joint">
+      <hardwareInterface>hardware_interface/PositionJointInterface</hardwareInterface>
+    </joint>
+    <actuator name="motor5">
+      <hardwareInterface>hardware_interface/PositionJointInterface</hardwareInterface>
+      <mechanicalReduction>1</mechanicalReduction>
+    </actuator>
+  </transmission>
+  <transmission name="tran6">
+    <type>transmission_interface/SimpleTransmission</type>
+    <joint name="right_rear_steering_joint">
+      <hardwareInterface>hardware_interface/PositionJointInterface</hardwareInterface>
+    </joint>
+    <actuator name="motor6">
+      <hardwareInterface>hardware_interface/PositionJointInterface</hardwareInterface>
+      <mechanicalReduction>1</mechanicalReduction>
+    </actuator>
+  </transmission>
+  <transmission name="tran7">
+    <type>transmission_interface/SimpleTransmission</type>
+    <joint name="left_front_wheel_joint">
+      <hardwareInterface>hardware_interface/VelocityJointInterface</hardwareInterface>
+    </joint>
+    <actuator name="motor7">
+      <hardwareInterface>hardware_interface/VelocityJointInterface</hardwareInterface>
+      <mechanicalReduction>1</mechanicalReduction>
+    </actuator>
+  </transmission>
+  <transmission name="tran8">
+    <type>transmission_interface/SimpleTransmission</type>
+    <joint name="right_front_wheel_joint">
+      <hardwareInterface>hardware_interface/VelocityJointInterface</hardwareInterface>
+    </joint>
+    <actuator name="motor8">
+      <hardwareInterface>hardware_interface/VelocityJointInterface</hardwareInterface>
+      <mechanicalReduction>1</mechanicalReduction>
+    </actuator>
+  </transmission>
+  <!-- Transmission for front wheels -->
+  <!--
+  <transmission name="tran5">
+    <type>transmission_interface/SimpleTransmission</type>
+    <joint name="left_front_wheel_joint">
+      <hardwareInterface>hardware_interface/VelocityJointInterface</hardwareInterface>
+    </joint>
+    <actuator name="motor5">
+      <hardwareInterface>hardware_interface/VelocityJointInterface</hardwareInterface>
+      <mechanicalReduction>1</mechanicalReduction>
+    </actuator>
+  </transmission>
+  <transmission name="tran6">
+    <type>transmission_interface/SimpleTransmission</type>
+    <joint name="right_front_wheel_joint">
+      <hardwareInterface>hardware_interface/VelocityJointInterface</hardwareInterface>
+    </joint>
+    <actuator name="motor6">
+      <hardwareInterface>hardware_interface/VelocityJointInterface</hardwareInterface>
+      <mechanicalReduction>1</mechanicalReduction>
+    </actuator>
+  </transmission> -->
+  <!--
+  <gazebo>
+    <plugin name="differential_drive_controller" filename="libgazebo_ros_diff_drive.so">
+      <robotNamespace>/</robotNamespace>
+      <alwaysOn>false</alwaysOn>
+      <updateRate>100</updateRate>
+      <leftJoint>left_rear_wheel_joint</leftJoint>
+      <rightJoint>right_rear_wheel_joint</rightJoint>
+      <wheelSeparation>1.0</wheelSeparation>
+      <wheelDiameter>0.4</wheelDiameter>
+      <torque>20</torque>
+      <commandTopic>cmd_vel</commandTopic>
+      <odometryTopic>asc/odom</odometryTopic>
+      <odometryFrame>map</odometryFrame>
+      <robotBaseFrame>base_link</robotBaseFrame>
+      <legacyMode>false</legacyMode>
+      <rosDebugLevel>Debug</rosDebugLevel>
+      <publishWheelTF>true</publishWheelTF>
+      <publishWheelJointState>true</publishWheelJointState>
+      <wheelAcceleration>5</wheelAcceleration>
+      <wheelTorque>20</wheelTorque>
+      <publishTf>1</publishTf>
+      <odometrySource>encoder</odometrySource>
+    </plugin>
+  </gazebo>-->
+  <!-- Extra joints for defining middle for the ackermann steering -->
 </robot>

Commit message: b4 adding move_base

File: asc_description/urdf/asc.urdf.xacro (robot description, xacro)
@@ -1,4 +1,4 @@
 <?xml version="1.0"?>
-<robot xmlns:xacro="http://www.ros.org/wiki/xacro" name="robot">
+<robot xmlns:xacro="http://www.ros.org/wiki/xacro" name="asc">
   <gazebo>
     <plugin name="gazebo_ros_control" filename="libgazebo_ros_control.so">
@@ -308,51 +308,8 @@
     </actuator>
   </transmission>
-  <!-- Transmission for front wheels -->
-  <!--
-  <transmission name="tran5">
-    <type>transmission_interface/SimpleTransmission</type>
-    <joint name="left_front_wheel_joint">
-      <hardwareInterface>hardware_interface/VelocityJointInterface</hardwareInterface>
-    </joint>
-    <actuator name="motor5">
-      <hardwareInterface>hardware_interface/VelocityJointInterface</hardwareInterface>
-      <mechanicalReduction>1</mechanicalReduction>
-    </actuator>
-  </transmission>
-  <transmission name="tran6">
-    <type>transmission_interface/SimpleTransmission</type>
-    <joint name="right_front_wheel_joint">
-      <hardwareInterface>hardware_interface/VelocityJointInterface</hardwareInterface>
-    </joint>
-    <actuator name="motor6">
-      <hardwareInterface>hardware_interface/VelocityJointInterface</hardwareInterface>
-      <mechanicalReduction>1</mechanicalReduction>
-    </actuator>
-  </transmission> -->
-  <!--
-  <gazebo>
-    <plugin name="differential_drive_controller" filename="libgazebo_ros_diff_drive.so">
-      <robotNamespace>/</robotNamespace>
-      <alwaysOn>false</alwaysOn>
-      <updateRate>100</updateRate>
-      <leftJoint>left_rear_wheel_joint</leftJoint>
-      <rightJoint>right_rear_wheel_joint</rightJoint>
-      <wheelSeparation>1.0</wheelSeparation>
-      <wheelDiameter>0.4</wheelDiameter>
-      <torque>20</torque>
-      <commandTopic>cmd_vel</commandTopic>
-      <odometryTopic>asc/odom</odometryTopic>
-      <odometryFrame>map</odometryFrame>
-      <robotBaseFrame>base_link</robotBaseFrame>
-      <legacyMode>false</legacyMode>
-      <rosDebugLevel>Debug</rosDebugLevel>
-      <publishWheelTF>true</publishWheelTF>
-      <publishWheelJointState>true</publishWheelJointState>
-      <wheelAcceleration>5</wheelAcceleration>
-      <wheelTorque>20</wheelTorque>
-      <publishTf>1</publishTf>
-      <odometrySource>encoder</odometrySource>
-    </plugin>
-  </gazebo>-->
-  <!-- Extra joints for defining middle for the ackermann steering -->
+<!-- Sensors -->
+  <xacro:include filename="$(find velodyne_description)/urdf/VLP-16.urdf.xacro"/>
+  <VLP-16 parent="frame_link" name="velodyne" topic="/velodyne_points" hz="10" samples="440" gpu="false">
+    <origin xyz="0 0 0.5" rpy="0 0 0" />
+  </VLP-16>
 </robot>

Commit message: need to fix config for cartographer

File: asc_description/urdf/asc.urdf.xacro (robot description, xacro)
@@ -3,5 +3,5 @@
   <gazebo>
     <plugin name="gazebo_ros_control" filename="libgazebo_ros_control.so">
-      <robotNamespace>/asc</robotNamespace>
+      <robotNamespace>/</robotNamespace>
       <!--<robotParam>/robot_description</robotParam> -->
       <robotSimType>gazebo_ros_control/DefaultRobotHWSim</robotSimType>
@@ -10,8 +10,7 @@
   <link name="base_link"/>
   <joint name="base_link_to_frame" type="fixed">
-    <origin xyz="0 0 1" rpy="0 0 0"/>
+    <origin xyz="0 0 0.7" rpy="0 0 0"/>
     <parent link="base_link"/>
     <child link="frame_link"/>
-    <axis xyz="0 0 1"/>
   </joint>
   <link name="frame_link">
@@ -310,6 +309,6 @@
 <!-- Sensors -->
   <xacro:include filename="$(find velodyne_description)/urdf/VLP-16.urdf.xacro"/>
-  <VLP-16 parent="frame_link" name="velodyne" topic="/velodyne_points" hz="10" samples="440" gpu="false">
-    <origin xyz="0 0 0.5" rpy="0 0 0" />
+  <VLP-16 parent="base_link" name="velodyne" topic="/velodyne_points" hz="10" samples="440" gpu="false">
+    <origin xyz="-0.45 0 1.15" rpy="0 0 0" />
   </VLP-16>
 </robot>

Commit message: added cartographer, works somewhat. Need to fix Odometry in four wheel steering  controller

File: asc_description/urdf/asc.urdf.xacro (robot description, xacro)
@@ -307,8 +307,22 @@
     </actuator>
   </transmission>
-<!-- Sensors -->
+  <!-- Sensors -->
+  <gazebo>
+    <plugin name="imu_controller" filename="libhector_gazebo_ros_imu.so">
+      <robotNamespace>/</robotNamespace>
+      <updateRate>50.0</updateRate>
+      <bodyName>base_link</bodyName>
+      <topicName>imu/data</topicName>
+      <accelDrift>0.005 0.005 0.005</accelDrift>
+      <accelGaussianNoise>0.005 0.005 0.005</accelGaussianNoise>
+      <rateDrift>0.005 0.005 0.005 </rateDrift>
+      <rateGaussianNoise>0.005 0.005 0.005 </rateGaussianNoise>
+      <headingDrift>0.005</headingDrift>
+      <headingGaussianNoise>0.005</headingGaussianNoise>
+    </plugin>
+  </gazebo>
   <xacro:include filename="$(find velodyne_description)/urdf/VLP-16.urdf.xacro"/>
   <VLP-16 parent="base_link" name="velodyne" topic="/velodyne_points" hz="10" samples="440" gpu="false">
-    <origin xyz="-0.45 0 1.15" rpy="0 0 0" />
+    <origin xyz="-0.45 0 1.15" rpy="0 0 0"/>
   </VLP-16>
 </robot>

Commit message: minor fixes, rtabmap not behaving as planned

File: asc_description/urdf/asc.urdf.xacro (robot description, xacro)
@@ -333,4 +333,63 @@
     </plugin>
   </gazebo>
+  <!-- add camera -->
+  <gazebo reference="camera_link">
+    <sensor type="depth" name="openni_camera_camera">
+      <always_on>1</always_on>
+      <visualize>true</visualize>
+      <camera>
+        <horizontal_fov>1.3962634</horizontal_fov>
+        <image>
+          <width>640</width>
+          <height>480</height>
+          <format>R8G8B8</format>
+        </image>
+        <clip>
+          <near>0.1</near>
+          <far>100</far>
+        </clip>
+      </camera>
+      <plugin name="camera_plugin" filename="libgazebo_ros_openni_kinect.so">
+        <baseline>0.2</baseline>
+        <alwaysOn>true</alwaysOn>
+        <!-- Keep this zero, update_rate in the parent <sensor> tag
+            will control the frame rate. -->
+        <updateRate>0.0</updateRate>
+        <cameraName>camera_ir</cameraName>
+        <imageTopicName>/camera/color/image_raw</imageTopicName>
+        <cameraInfoTopicName>/camera/color/camera_info</cameraInfoTopicName>
+        <depthImageTopicName>/camera/depth/image_raw</depthImageTopicName>
+        <depthImageCameraInfoTopicName>/camera/depth/camera_info</depthImageCameraInfoTopicName>
+        <pointCloudTopicName>/camera/depth/points</pointCloudTopicName>
+        <frameName>camera_link</frameName>
+        <pointCloudCutoff>0.5</pointCloudCutoff>
+        <pointCloudCutoffMax>3.0</pointCloudCutoffMax>
+        <distortionK1>0</distortionK1>
+        <distortionK2>0</distortionK2>
+        <distortionK3>0</distortionK3>
+        <distortionT1>0</distortionT1>
+        <distortionT2>0</distortionT2>
+        <CxPrime>0</CxPrime>
+        <Cx>0</Cx>
+        <Cy>0</Cy>
+        <focalLength>0</focalLength>
+        <hackBaseline>0</hackBaseline>
+      </plugin>
+    </sensor>
+  </gazebo>
+  <link name="camera_link"/>
+  <!--
+  <link name="cameraLeft_depth_link"/> -->
+  <joint name="cameraLeft_joint" type="fixed">
+    <origin xyz="0 0 1" rpy="0 0.1 0"/>
+    <parent link="base_link"/>
+    <child link="camera_link"/>
+  </joint>
+  <!--
+  <joint name="cameraLeft_depth_joint" type="fixed">
+    <origin xyz="0 0 0" rpy="-1.57 0 -1.57"/>
+    <parent link="camera_link"/>
+    <child link="camera_link_depth_link"/>
+  </joint> -->
   <xacro:include filename="$(find velodyne_description)/urdf/VLP-16.urdf.xacro"/>
   <VLP-16 parent="base_link" name="velodyne" topic="/velodyne_points" hz="10" samples="440" gpu="false">

Commit message: clean-up for depends in xml files

File: asc_description/urdf/asc.urdf.xacro (robot description, xacro)
@@ -382,5 +382,5 @@
   <link name="cameraLeft_depth_link"/> -->
   <joint name="cameraLeft_joint" type="fixed">
-    <origin xyz="0 0 1" rpy="0 0.1 0"/>
+    <origin xyz="0 3 1" rpy="0 0.1 0"/>
     <parent link="base_link"/>
     <child link="camera_link"/>
