Commit message: use_odom apparently solved a lot of problems...

File: asc_description/urdf/asc.urdf.xacro (robot description, xacro)
@@ -6,4 +6,5 @@
       <!--<robotParam>/robot_description</robotParam> -->
       <robotSimType>gazebo_ros_control/DefaultRobotHWSim</robotSimType>
+      <legacyModeNS>false</legacyModeNS>
     </plugin>
   </gazebo>
@@ -314,4 +315,11 @@
       <bodyName>base_link</bodyName>
       <topicName>imu/data</topicName>
+      <accelDrift>0.00 0.00 0.00</accelDrift>
+      <accelGaussianNoise>0.00 0.00 0.00</accelGaussianNoise>
+      <rateDrift>0.0 0.000.0 </rateDrift>
+      <rateGaussianNoise>0.00 0.005 0.00 </rateGaussianNoise>
+      <headingDrift>0.00</headingDrift>
+      <headingGaussianNoise>0.00</headingGaussianNoise>
+      <!--
       <accelDrift>0.005 0.005 0.005</accelDrift>
       <accelGaussianNoise>0.005 0.005 0.005</accelGaussianNoise>
@@ -319,16 +327,40 @@
       <rateGaussianNoise>0.005 0.005 0.005 </rateGaussianNoise>
       <headingDrift>0.005</headingDrift>
-      <headingGaussianNoise>0.005</headingGaussianNoise>
+      <headingGaussianNoise>0.005</headingGaussianNoise> -->
     </plugin>
     <!-- for calculating perfect odometry -->
+    <!--
     <plugin name="p3d_base_controller" filename="libgazebo_ros_p3d.so">
       <alwaysOn>true</alwaysOn>
-      <updateRate>50.0</updateRate>
+      <updateRate>1.0</updateRate>
       <bodyName>base_link</bodyName>
-      <topicName>odom_perfect</topicName>
+      <topicName>odom_perfect_world</topicName>
       <gaussianNoise>0.0</gaussianNoise>
       <frameName>world</frameName>
       <xyzOffsets>0 0 0</xyzOffsets>
       <rpyOffsets>0 0 0</rpyOffsets>
+    </plugin>
+    <link name="odom"/>
+    <plugin name="p3d_base_controller" filename="libgazebo_ros_p3d.so">
+      <alwaysOn>true</alwaysOn>
+      <updateRate>1.0</updateRate>
+      <bodyName>base_link</bodyName>
+      <topicName>odom_perfect</topicName>
+      <gaussianNoise>0.0</gaussianNoise>
+      <frameName>odom</frameName>
+      <xyzOffsets>0 0 0</xyzOffsets>
+      <rpyOffsets>0 0 0</rpyOffsets>
+    </plugin> -->
+    <!-- add gps -->
+    <plugin name="gps_sim" filename="libhector_gazebo_ros_gps.so">
+      <alwaysOn>1</alwaysOn>
+      <updateRate>10.0</updateRate>
+      <bodyName>base_link</bodyName>
+      <topicName>fix</topicName>
+      <velocityTopicName>fix_velocity</velocityTopicName>
+      <drift>5.0 5.0 5.0</drift>
+      <gaussianNoise>0.1 0.1 0.1</gaussianNoise>
+      <velocityDrift>0 0 0</velocityDrift>
+      <velocityGaussianNoise>0.1 0.1 0.1</velocityGaussianNoise>
     </plugin>
   </gazebo>
@@ -362,5 +394,5 @@
         <depthImageCameraInfoTopicName>/camera/depth/camera_info</depthImageCameraInfoTopicName>
         <pointCloudTopicName>/camera/depth/points</pointCloudTopicName>
-        <frameName>camera_link</frameName>
+        <frameName>camera_link_pc</frameName>
         <pointCloudCutoff>0.5</pointCloudCutoff>
         <pointCloudCutoffMax>3.0</pointCloudCutoffMax>
@@ -381,15 +413,15 @@
   <!--
   <link name="cameraLeft_depth_link"/> -->
-  <joint name="cameraLeft_joint" type="fixed">
-    <origin xyz="0 3 1" rpy="0 0.1 0"/>
+  <joint name="base_to_camera" type="fixed">
+    <origin xyz="1.2 0 0.6" rpy="0 0.1 0"/>
     <parent link="base_link"/>
     <child link="camera_link"/>
   </joint>
-  <!--
-  <joint name="cameraLeft_depth_joint" type="fixed">
+  <link name="camera_link_pc"/>
+  <joint name="camera_to_pc" type="fixed">
     <origin xyz="0 0 0" rpy="-1.57 0 -1.57"/>
     <parent link="camera_link"/>
-    <child link="camera_link_depth_link"/>
-  </joint> -->
+    <child link="camera_link_pc"/>
+  </joint>
   <xacro:include filename="$(find velodyne_description)/urdf/VLP-16.urdf.xacro"/>
   <VLP-16 parent="base_link" name="velodyne" topic="/velodyne_points" hz="10" samples="440" gpu="false">

Commit message: adjusted gazebo model to use topic names of real launch file

File: asc_description/urdf/asc.urdf.xacro (robot description, xacro)
@@ -315,4 +315,5 @@
       <bodyName>base_link</bodyName>
       <topicName>imu/data</topicName>
+      <!--
       <accelDrift>0.00 0.00 0.00</accelDrift>
       <accelGaussianNoise>0.00 0.00 0.00</accelGaussianNoise>
@@ -320,6 +321,5 @@
       <rateGaussianNoise>0.00 0.005 0.00 </rateGaussianNoise>
       <headingDrift>0.00</headingDrift>
-      <headingGaussianNoise>0.00</headingGaussianNoise>
-      <!--
+      <headingGaussianNoise>0.00</headingGaussianNoise> -->
       <accelDrift>0.005 0.005 0.005</accelDrift>
       <accelGaussianNoise>0.005 0.005 0.005</accelGaussianNoise>
@@ -327,5 +327,5 @@
       <rateGaussianNoise>0.005 0.005 0.005 </rateGaussianNoise>
       <headingDrift>0.005</headingDrift>
-      <headingGaussianNoise>0.005</headingGaussianNoise> -->
+      <headingGaussianNoise>0.005</headingGaussianNoise>
     </plugin>
     <!-- for calculating perfect odometry -->
@@ -391,12 +391,12 @@
         <updateRate>0.0</updateRate>
         <cameraName>camera_ir</cameraName>
-        <imageTopicName>/camera/color/image_raw</imageTopicName>
-        <cameraInfoTopicName>/camera/color/camera_info</cameraInfoTopicName>
-        <depthImageTopicName>/camera/depth/image_raw</depthImageTopicName>
-        <depthImageCameraInfoTopicName>/camera/depth/camera_info</depthImageCameraInfoTopicName>
-        <pointCloudTopicName>/camera/depth/points</pointCloudTopicName>
+        <imageTopicName>/zed/zed_node/rgb/image_rect_color</imageTopicName>
+        <cameraInfoTopicName>/zed/zed_node/rgb/camera_info </cameraInfoTopicName>
+        <depthImageTopicName>/zed/zed_node/depth/depth_registered</depthImageTopicName>
+        <depthImageCameraInfoTopicName>/zed/zed_node/depth/image_raw/camera_info</depthImageCameraInfoTopicName>
+        <pointCloudTopicName>/zed/zed_node/point_cloud/cloud_registered </pointCloudTopicName>
         <frameName>camera_link_pc</frameName>
         <pointCloudCutoff>0.4</pointCloudCutoff>
-        <!--
+        <!-- does nothing it seems
         <pointCloudCutoffMax>20.0</pointCloudCutoffMax> -->
         <distortionK1>0</distortionK1>
@@ -414,6 +414,4 @@
   </gazebo>
   <link name="camera_link"/>
-  <!--
-  <link name="cameraLeft_depth_link"/> -->
   <joint name="base_to_camera" type="fixed">
     <origin xyz="1.2 0 0.6" rpy="0 0.1 0"/>
@@ -428,5 +426,5 @@
   </joint>
   <xacro:include filename="$(find velodyne_description)/urdf/VLP-16.urdf.xacro"/>
-  <VLP-16 parent="base_link" name="velodyne" topic="/velodyne_points" hz="10" samples="440" gpu="false">
+  <VLP-16 parent="base_link" name="velodyne" topic="/os1_cloud_node/points" hz="10" samples="440" gpu="false">
     <origin xyz="-0.45 0 1.15" rpy="0 0 0"/>
   </VLP-16>

Commit message: trying to resolve rtab for simulation

File: asc_description/urdf/asc.urdf.xacro (robot description, xacro)
@@ -11,5 +11,5 @@
   <link name="base_link"/>
   <joint name="base_link_to_frame" type="fixed">
-    <origin xyz="0 0 0.7" rpy="0 0 0"/>
+    <origin xyz="0 0 0.6" rpy="0 0 0"/>
     <parent link="base_link"/>
     <child link="frame_link"/>

Commit message: minor tuning to teb parameters

File: asc_description/urdf/asc.urdf.xacro (robot description, xacro)
@@ -11,5 +11,5 @@
   <link name="base_link"/>
   <joint name="base_link_to_frame" type="fixed">
-    <origin xyz="0 0 0.6" rpy="0 0 0"/>
+    <origin xyz="0 0 0.7" rpy="0 0 0"/>
     <parent link="base_link"/>
     <child link="frame_link"/>
