Commit message: added new model, deprecated old solarcar urdf, saved as sc_description

File: asc_description/urdf/asc.urdf.xacro (robot description, xacro)
@@ -1,4 +1,6 @@
-<?xml version="1.0"?>
-<robot xmlns:xacro="http://www.ros.org/wiki/xacro" name="asc">
+<?xml version="1.0" encoding="utf-8"?>
+<robot xmlns:xacro="http://www.ros.org/wiki/xacro"
+  name="asc">
+  <xacro:arg name="simulation" default="true" />
   <gazebo>
     <plugin name="gazebo_ros_control" filename="libgazebo_ros_control.so">
@@ -9,7 +11,12 @@
     </plugin>
   </gazebo>
+  <xacro:include filename="macro_link.urdf.xacro"/>
+  <xacro:include filename="macro_wheel.urdf.xacro"/>
+  <xacro:property name="wheel_length" value="0.032"/>
+  <xacro:property name="wheel_radius" value="0.1"/>
+  <xacro:property name="wheel_parent" value="frame_link"/>
   <link name="base_link"/>
   <joint name="base_link_to_frame" type="fixed">
-    <origin xyz="0 0 0.7" rpy="0 0 0"/>
+    <origin xyz="0 0 0" rpy="0 0 0"/>
     <parent link="base_link"/>
     <child link="frame_link"/>
@@ -24,5 +31,5 @@
       <origin xyz="0 0 0" rpy="0 0 0"/>
       <geometry>
-        <mesh filename="package://asc_description/meshes/base_link.STL"/>
+        <mesh filename="package://asc_description/meshes/base_link.STL" />
       </geometry>
       <material name="">
@@ -30,283 +37,49 @@
       </material>
     </visual>
-    <!--
-    <collision>
-      <origin xyz="0 0 0" rpy="0 0 0"/>
-      <geometry>
-        <mesh filename="package://asc_description/meshes/base_link.STL"/>
-      </geometry>
-    </collision> -->
   </link>
-  <link name="left_front_steering_link">
-    <inertial>
-      <origin xyz="-0.0439194980427094 -0.0123148656628935 -0.29574701698731" rpy="0 0 0"/>
-      <mass value="5.71439015182903"/>
-      <inertia ixx="0.138973038944984" ixy="0.00240438901312515" ixz="0.0320681563279578" iyy="0.160053837434921" iyz="-0.0109556260035955" izz="0.028546837728721"/>
-    </inertial>
-    <visual>
-      <origin xyz="0 0 0" rpy="0 0 0"/>
-      <geometry>
-        <mesh filename="package://asc_description/meshes/left_front_steering_link.STL"/>
-      </geometry>
-      <material name="">
-        <color rgba="0.792156862745098 0.819607843137255 0.933333333333333 1"/>
-      </material>
-    </visual>
-    <collision>
-      <origin xyz="0 0 0" rpy="0 0 0"/>
-      <geometry>
-        <mesh filename="package://asc_description/meshes/left_front_steering_link.STL"/>
-      </geometry>
-    </collision>
-  </link>
-  <joint name="left_front_steering_joint" type="revolute">
-    <origin xyz="0.9825 0.63618 0.047063" rpy="0.13546 -0.28749 0.0037802"/>
-    <parent link="frame_link"/>
-    <child link="left_front_steering_link"/>
-    <axis xyz="0 0 1"/>
-    <limit lower="-0.8" upper="0.9" effort="100" velocity="100"/>
-  </joint>
-  <link name="left_front_wheel_link">
-    <inertial>
-      <origin xyz="-2.26485497023532E-14 4.10782519111308E-14 0.00509989314954018" rpy="0 0 0"/>
-      <mass value="3.6905479088754"/>
-      <inertia ixx="0.117114266308146" ixy="-6.93889390390723E-18" ixz="1.02756637900478E-17" iyy="0.117114266308146" iyz="-3.62378420062206E-17" izz="0.227951064044091"/>
-    </inertial>
-    <visual>
-      <origin xyz="0 0 0" rpy="0 0 0"/>
-      <geometry>
-        <cylinder length="0.05" radius="0.3"/>
-      </geometry>
-    </visual>
-    <collision>
-      <origin xyz="0 0 0" rpy="0 0 0"/>
-      <geometry>
-        <cylinder length="0.05" radius="0.3"/>
-      </geometry>
-    </collision>
-  </link>
-  <joint name="left_front_wheel_joint" type="continuous">
-    <origin xyz="0.065693 0.065054 -0.50813" rpy="-1.8471 1.0585 -0.24589"/>
-    <parent link="left_front_steering_link"/>
-    <child link="left_front_wheel_link"/>
-    <axis xyz="0 0 1"/>
-  </joint>
-  <link name="right_front_steering_link">
-    <inertial>
-      <origin xyz="-0.0465182122250822 0.0145095544427134 -0.290619703564971" rpy="0 0 0"/>
-      <mass value="5.57746367002881"/>
-      <inertia ixx="0.138857493635095" ixy="-0.0022557465179349" ixz="0.032139397456901" iyy="0.160001336296301" iyz="0.0107272499121531" izz="0.0284811002523076"/>
-    </inertial>
-    <visual>
-      <origin xyz="0 0 0" rpy="0 0 0"/>
-      <geometry>
-        <mesh filename="package://asc_description/meshes/right_front_steering_link.STL"/>
-      </geometry>
-      <material name="">
-        <color rgba="0.792156862745098 0.819607843137255 0.933333333333333 1"/>
-      </material>
-    </visual>
-    <collision>
-      <origin xyz="0 0 0" rpy="0 0 0"/>
-      <geometry>
-        <mesh filename="package://asc_description/meshes/right_front_steering_link.STL"/>
-      </geometry>
-    </collision>
-  </link>
-  <joint name="right_front_steering_joint" type="revolute">
-    <origin xyz="0.9825 -0.63318 0.047063" rpy="-0.13546 -0.28749 0.0037802"/>
-    <parent link="frame_link"/>
-    <child link="right_front_steering_link"/>
-    <axis xyz="0 0 1"/>
-    <limit lower="-0.8" upper="0.8" effort="100" velocity="100"/>
-  </joint>
-  <link name="right_front_wheel_link">
-    <inertial>
-      <origin xyz="-1.02140518265514E-14 6.85007606193722E-14 0.00509989314946457" rpy="0 0 0"/>
-      <mass value="3.69054790887537"/>
-      <inertia ixx="0.117114266308143" ixy="1.38777878078145E-17" ixz="2.37549730750149E-18" iyy="0.117114266308143" iyz="3.40770700491441E-17" izz="0.22795106404409"/>
-    </inertial>
-    <visual>
-      <origin xyz="0 0 0" rpy="0 0 0"/>
-      <geometry>
-        <cylinder length="0.05" radius="0.3"/>
-      </geometry>
-    </visual>
-    <collision>
-      <origin xyz="0 0 0" rpy="0 0 0"/>
-      <geometry>
-        <cylinder length="0.05" radius="0.3"/>
-      </geometry>
-    </collision>
-  </link>
-  <joint name="right_front_wheel_joint" type="continuous">
-    <origin xyz="0.065291 -0.059582 -0.50741" rpy="1.8455 1.0552 0.23683"/>
-    <parent link="right_front_steering_link"/>
-    <child link="right_front_wheel_link"/>
-    <axis xyz="0 0 1"/>
-  </joint>
-  <!-- add fake rear steering joint-->
-  <link name="left_rear_steer">
-    <inertial>
-      <origin xyz="0 0 0" rpy="0 0 0"/>
-      <mass value="1"/>
-      <inertia ixx="1.0" ixy="0.0" ixz="0.0" iyy="1.0" iyz="0.0" izz="1.0"/>
-    </inertial>
-  </link>
-  <joint name="left_rear_steering_joint" type="revolute">
-    <origin xyz="-1.3237 0.70906 -0.41261" rpy="0 0 0"/>
-    <parent link="frame_link"/>
-    <child link="left_rear_steer"/>
-    <axis xyz="0 0 1"/>
-    <limit lower="0" upper="0" effort="0" velocity="0"/>
-  </joint>
-  <link name="left_rear_wheel">
-    <inertial>
-      <origin xyz="8.43769498715119E-15 0.0589722640664191 -5.01820807130571E-14" rpy="0 0 0"/>
-      <mass value="3.68939811577995"/>
-      <inertia ixx="0.117113236563891" ixy="-4.42261767048626E-17" ixz="-6.93889390390723E-18" iyy="0.227950884881602" iyz="-3.11187820789416E-16" izz="0.117113236563891"/>
-    </inertial>
-    <visual>
-      <origin xyz="0 0 0" rpy="1.57 0 0"/>
-      <geometry>
-        <cylinder length="0.05" radius="0.3"/>
-      </geometry>
-    </visual>
-    <collision>
-      <origin xyz="0 0 0" rpy="1.57 0 0"/>
-      <geometry>
-        <cylinder length="0.05" radius="0.3"/>
-      </geometry>
-    </collision>
-  </link>
-  <joint name="left_rear_wheel_joint" type="continuous">
-    <origin xyz="0 0 0" rpy="0 0 0"/>
-    <parent link="left_rear_steer"/>
-    <child link="left_rear_wheel"/>
-    <axis xyz="0 1 0"/>
-  </joint>
-  <!-- add fake rear steering joint-->
-  <link name="right_rear_steer">
-    <inertial>
-      <origin xyz="0 0 0" rpy="0 0 0"/>
-      <mass value="1"/>
-      <inertia ixx="1.0" ixy="0.0" ixz="0.0" iyy="1.0" iyz="0.0" izz="1.0"/>
-    </inertial>
-  </link>
-  <joint name="right_rear_steering_joint" type="revolute">
-    <origin xyz="-1.3237 -0.70606 -0.41261" rpy="0 0 0"/>
-    <parent link="frame_link"/>
-    <child link="right_rear_steer"/>
-    <axis xyz="0 0 1"/>
-    <limit lower="0" upper="0" effort="0" velocity="0"/>
-  </joint>
-  <link name="right_rear_wheel">
-    <inertial>
-      <origin xyz="7.99360577730113E-15 0.0589722640664192 4.2410519540681E-14" rpy="0 0 0"/>
-      <mass value="3.68939811577991"/>
-      <inertia ixx="0.117113236563893" ixy="-4.66966016159301E-17" ixz="4.33680868994202E-18" iyy="0.2279508848816" iyz="3.34438350256477E-16" izz="0.117113236563893"/>
-    </inertial>
-    <visual>
-      <origin xyz="0 0 0" rpy="1.57 0 0"/>
-      <geometry>
-        <cylinder length="0.05" radius="0.3"/>
-      </geometry>
-    </visual>
-    <collision>
-      <origin xyz="0 0 0" rpy="1.57 0 0"/>
-      <geometry>
-        <cylinder length="0.05" radius="0.3"/>
-      </geometry>
-    </collision>
-  </link>
-  <joint name="right_rear_wheel_joint" type="continuous">
-    <origin xyz="0 0 0" rpy="0 0 0"/>
-    <parent link="right_rear_steer"/>
-    <child link="right_rear_wheel"/>
-    <axis xyz="0 1 0"/>
-  </joint>
-  <transmission name="tran1">
-    <type>transmission_interface/SimpleTransmission</type>
-    <joint name="left_rear_wheel_joint">
-      <hardwareInterface>hardware_interface/VelocityJointInterface</hardwareInterface>
-    </joint>
-    <actuator name="motor1">
-      <hardwareInterface>hardware_interface/VelocityJointInterface</hardwareInterface>
-      <mechanicalReduction>1</mechanicalReduction>
-    </actuator>
-  </transmission>
-  <transmission name="tran2">
-    <type>transmission_interface/SimpleTransmission</type>
-    <joint name="right_rear_wheel_joint">
-      <hardwareInterface>hardware_interface/VelocityJointInterface</hardwareInterface>
-    </joint>
-    <actuator name="motor2">
-      <hardwareInterface>hardware_interface/VelocityJointInterface</hardwareInterface>
-      <mechanicalReduction>1</mechanicalReduction>
-    </actuator>
-  </transmission>
-  <!-- Transmissions for steering joints-->
-  <transmission name="tran3">
-    <type>transmission_interface/SimpleTransmission</type>
-    <joint name="left_front_steering_joint">
-      <hardwareInterface>hardware_interface/PositionJointInterface</hardwareInterface>
-    </joint>
-    <actuator name="motor3">
-      <hardwareInterface>hardware_interface/PositionJointInterface</hardwareInterface>
-      <mechanicalReduction>1</mechanicalReduction>
-    </actuator>
-  </transmission>
-  <transmission name="tran4">
-    <type>transmission_interface/SimpleTransmission</type>
-    <joint name="right_front_steering_joint">
-      <hardwareInterface>hardware_interface/PositionJointInterface</hardwareInterface>
-    </joint>
-    <actuator name="motor4">
-      <hardwareInterface>hardware_interface/PositionJointInterface</hardwareInterface>
-      <mechanicalReduction>1</mechanicalReduction>
-    </actuator>
-  </transmission>
-  <!-- Transmissions for fake steering joints-->
-  <transmission name="tran5">
-    <type>transmission_interface/SimpleTransmission</type>
-    <joint name="left_rear_steering_joint">
-      <hardwareInterface>hardware_interface/PositionJointInterface</hardwareInterface>
-    </joint>
-    <actuator name="motor5">
-      <hardwareInterface>hardware_interface/PositionJointInterface</hardwareInterface>
-      <mechanicalReduction>1</mechanicalReduction>
-    </actuator>
-  </transmission>
-  <transmission name="tran6">
-    <type>transmission_interface/SimpleTransmission</type>
-    <joint name="right_rear_steering_joint">
-      <hardwareInterface>hardware_interface/PositionJointInterface</hardwareInterface>
-    </joint>
-    <actuator name="motor6">
-      <hardwareInterface>hardware_interface/PositionJointInterface</hardwareInterface>
-      <mechanicalReduction>1</mechanicalReduction>
-    </actuator>
-  </transmission>
-  <transmission name="tran7">
-    <type>transmission_interface/SimpleTransmission</type>
-    <joint name="left_front_wheel_joint">
-      <hardwareInterface>hardware_interface/VelocityJointInterface</hardwareInterface>
-    </joint>
-    <actuator name="motor7">
-      <hardwareInterface>hardware_interface/VelocityJointInterface</hardwareInterface>
-      <mechanicalReduction>1</mechanicalReduction>
-    </actuator>
-  </transmission>
-  <transmission name="tran8">
-    <type>transmission_interface/SimpleTransmission</type>
-    <joint name="right_front_wheel_joint">
-      <hardwareInterface>hardware_interface/VelocityJointInterface</hardwareInterface>
-    </joint>
-    <actuator name="motor8">
-      <hardwareInterface>hardware_interface/VelocityJointInterface</hardwareInterface>
-      <mechanicalReduction>1</mechanicalReduction>
-    </actuator>
-  </transmission>
-  <!-- Sensors -->
+  <xacro:asc_wheel_front wheel_prefix="right"
+  link_parent="${wheel_parent}" wheel_length="${wheel_length}" wheel_radius="${wheel_radius}" >
+    <origin
+      xyz="0.35635 -0.23074 0.27672"
+      rpy="0.29046 -0.12882 -1.6092" />
+    <origin
+      xyz="0.024 0.023741 -0.18704"
+      rpy="0.13981 0.28531 1.6105" />
+    <axis
+      xyz="5.3677E-05 1 0.00055924" />
+  </xacro:asc_wheel_front>
+  <xacro:asc_wheel_front wheel_prefix="left"
+  link_parent="${wheel_parent}" wheel_length="${wheel_length}" wheel_radius="${wheel_radius}" >
+    <origin
+      xyz="0.35635 0.22966 0.274"
+      rpy="0.28907 0.00024223 -1.5707" />
+    <origin
+      xyz="-0.05 0.023546 -0.17951"
+      rpy="1.5963E-05 0.28907 1.5707" />
+    <axis
+      xyz="5.3677E-05 -1 0.00055924" />
+  </xacro:asc_wheel_front>
+  <xacro:asc_wheel_rear wheel_prefix="right"
+  link_parent="${wheel_parent}" wheel_length="${wheel_length}" wheel_radius="${wheel_radius}" >
+  <origin
+  xyz="-0.48012 -0.29752 0.27"
+  rpy="0.0 0.0 0.0" />
+    <origin
+      xyz="0.0 0.0 -0.16"
+      rpy="0 0 0" />
+    <axis
+      xyz="0 1 0" />
+  </xacro:asc_wheel_rear>
+  <xacro:asc_wheel_rear wheel_prefix="left"
+  link_parent="${wheel_parent}" wheel_length="${wheel_length}" wheel_radius="${wheel_radius}" >
+  <origin
+  xyz="-0.48012 0.29752 0.27"
+  rpy="0.0 0.0 0.0" />
+      <origin
+      xyz="0.0 0.0 -0.16"
+      rpy="0 0 0" />
+    <axis
+      xyz="0 1 0" />
+  </xacro:asc_wheel_rear>
   <gazebo>
     <plugin name="imu_controller" filename="libhector_gazebo_ros_imu.so">
@@ -315,11 +88,4 @@
       <bodyName>base_link</bodyName>
       <topicName>imu/data</topicName>
-      <!--
-      <accelDrift>0.00 0.00 0.00</accelDrift>
-      <accelGaussianNoise>0.00 0.00 0.00</accelGaussianNoise>
-      <rateDrift>0.0 0.000.0 </rateDrift>
-      <rateGaussianNoise>0.00 0.005 0.00 </rateGaussianNoise>
-      <headingDrift>0.00</headingDrift>
-      <headingGaussianNoise>0.00</headingGaussianNoise> -->
       <accelDrift>0.005 0.005 0.005</accelDrift>
       <accelGaussianNoise>0.005 0.005 0.005</accelGaussianNoise>
@@ -329,28 +95,4 @@
       <headingGaussianNoise>0.005</headingGaussianNoise>
     </plugin>
-    <!-- for calculating perfect odometry -->
-    <!--
-    <plugin name="p3d_base_controller" filename="libgazebo_ros_p3d.so">
-      <alwaysOn>true</alwaysOn>
-      <updateRate>1.0</updateRate>
-      <bodyName>base_link</bodyName>
-      <topicName>odom_perfect_world</topicName>
-      <gaussianNoise>0.0</gaussianNoise>
-      <frameName>world</frameName>
-      <xyzOffsets>0 0 0</xyzOffsets>
-      <rpyOffsets>0 0 0</rpyOffsets>
-    </plugin>
-    <link name="odom"/>
-    <plugin name="p3d_base_controller" filename="libgazebo_ros_p3d.so">
-      <alwaysOn>true</alwaysOn>
-      <updateRate>1.0</updateRate>
-      <bodyName>base_link</bodyName>
-      <topicName>odom_perfect</topicName>
-      <gaussianNoise>0.0</gaussianNoise>
-      <frameName>odom</frameName>
-      <xyzOffsets>0 0 0</xyzOffsets>
-      <rpyOffsets>0 0 0</rpyOffsets>
-    </plugin> -->
-    <!-- add gps -->
     <plugin name="gps_controller" filename="libhector_gazebo_ros_gps.so">
       <robotNamespace>/</robotNamespace>
@@ -413,4 +155,21 @@
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
File: asc_description/urdf/macro_link.urdf.xacro (robot description, xacro)
@@ -1,4 +1,4 @@
 <?xml version="1.0"?>
-<robot xmlns:xacro="http://ros.org/wiki/xacro" name="asc_link">
+<robot xmlns:xacro="http://www.ros.org/wiki/xacro" name="asc_link">
 	<xacro:macro name="asc_wheel" params="x_size y_size z_size">
 	<geometry>

File: asc_description/urdf/macro_wheel.urdf.xacro (robot description, xacro)
@@ -1,24 +1,144 @@
 <?xml version="1.0"?>
-<robot xmlns:xacro="http://ros.org/wiki/xacro" name="asc_wheel">
-  <xacro:macro name="asc_wheel" params="wheel_prefix link_parent *joint_pose *wheel_rotation">
-    <link name="${wheel_prefix}_wheel">
+<robot xmlns:xacro="http://www.ros.org/wiki/xacro" name="asc_wheel">
+  <xacro:macro name="asc_wheel" params="wheel_prefix link_parent wheel_length wheel_radius *wheel_joint_origin *wheel_joint_axis">
+    <link name="${wheel_prefix}_wheel_link">
+      <inertial>
+        <origin xyz="-1.02140518265514E-14 6.85007606193722E-14 0.00509989314946457" rpy="0 0 0"/>
+        <mass value="3.6905479088754"/>
+        <inertia ixx="0.117114266308143" ixy="1.38777878078145E-17" ixz="2.37549730750149E-18" iyy="0.117114266308143" iyz="3.40770700491441E-17" izz="0.22795106404409"/>
+      </inertial>
       <visual>
-        <insert_block name="joint_pose"/>
+        <origin
+          xyz="0 0 0"
+          rpy="1.57 0 0" />
+      <!--
+      <geometry>
+        <mesh filename="package://asc_description/meshes/wheel.STL" />
+      </geometry> -->
         <geometry>
           <cylinder length="${wheel_length}" radius="${wheel_radius}"/>
         </geometry>
+        <material
+          name="">
+          <color
+            rgba="1 1 1 1" />
+        </material>
       </visual>
       <collision>
-        <insert_block name="joint_pose"/>
+        <origin
+          xyz="0 0 0"
+          rpy="1.57 0 0" />
         <geometry>
-          <cylinder length="${wheel_length}" radius="${wheel_radius}"/>
+        <cylinder length="${wheel_length}" radius="${wheel_radius}"/>
         </geometry>
       </collision>
     </link>
-    <joint name="${wheel_prefix}_joint" type="continuous">
-      <insert_block name="joint_pose"/>
+    <joint name="${wheel_prefix}_wheel_joint" type="continuous">
+      <xacro:insert_block name="wheel_joint_origin"/>
+      <parent
+        link="${wheel_prefix}_steering_link" />
+      <child
+        link="${wheel_prefix}_wheel_link" />
+      <xacro:insert_block name="wheel_joint_axis"/>
+    </joint>
+    <transmission name="${wheel_prefix}_wheel_joint_tran">
+      <type>transmission_interface/SimpleTransmission</type>
+      <joint name="${wheel_prefix}_wheel_joint">
+        <hardwareInterface>hardware_interface/VelocityJointInterface</hardwareInterface>
+      </joint>
+      <actuator name="${wheel_prefix}_wheel_joint_motor">
+        <hardwareInterface>hardware_interface/VelocityJointInterface</hardwareInterface>
+        <mechanicalReduction>1</mechanicalReduction>
+      </actuator>
+    </transmission>
+    <transmission name="${wheel_prefix}_steering_tran">
+      <type>transmission_interface/SimpleTransmission</type>
+      <joint name="${wheel_prefix}_steering_joint">
+        <hardwareInterface>hardware_interface/PositionJointInterface</hardwareInterface>
+      </joint>
+      <actuator name="${wheel_prefix}_steering_motor">
+        <hardwareInterface>hardware_interface/PositionJointInterface</hardwareInterface>
+        <mechanicalReduction>1</mechanicalReduction>
+      </actuator>
+    </transmission>
+  </xacro:macro>
+  <xacro:macro name="asc_wheel_front" params="wheel_prefix link_parent wheel_length wheel_radius *steering_joint_pose *wheel_joint_origin *wheel_joint_axis">
+    <link name="front_${wheel_prefix}_steering_link">
+      <inertial>
+        <origin
+          xyz="0.0 0.0 0.0"
+          rpy="0 0 0" />
+          <mass value="5.71439015182903"/>
+        <inertia
+          ixx="0.00107634033140466"
+          ixy="1.51573650824965E-05"
+          ixz="-6.94838293881106E-05"
+          iyy="0.000914613440717638"
+          iyz="0.000195407309247701"
+          izz="0.000234021785961031" />
+      </inertial>
+      <visual>
+        <origin
+          xyz="0 0 0"
+          rpy="0 0 0" />
+        <geometry>
+          <mesh
+            filename="package://asc_description/meshes/front_${wheel_prefix}_steering_link.STL" />
+        </geometry>
+        <material
+          name="">
+          <color
+            rgba="0.792156862745098 0.819607843137255 0.933333333333333 1" />
+        </material>
+      </visual>
+    </link>
+  <!-- Add base of wheel macro -->
+    <xacro:asc_wheel wheel_prefix="front_${wheel_prefix}"
+    link_parent="${link_parent}" wheel_length="${wheel_length}" wheel_radius="${wheel_radius}" >
+    <xacro:insert_block name="wheel_joint_origin"/>
+    <xacro:insert_block name="wheel_joint_axis"/>
+    </xacro:asc_wheel>
+    <!-- Add specfic parts for forward wheels-->
+    <joint name="front_${wheel_prefix}_steering_joint" type="revolute">
+      <xacro:insert_block name="steering_joint_pose"/>
       <parent link="${link_parent}"/>
-      <child link="${wheel_prefix}_wheel"/>
-      <axis xyz="0 1 0"/>
+      <child link="front_${wheel_prefix}_steering_link"/>
+      <axis xyz="0 0 1"/>
+      <limit lower="-0.8" upper="0.9" effort="100" velocity="100"/>
+    </joint>
+  </xacro:macro>
+  <xacro:macro name="asc_wheel_rear" params="wheel_prefix link_parent wheel_length wheel_radius *steering_joint_pose *wheel_joint_origin *wheel_joint_axis">
+    <link name="rear_${wheel_prefix}_steering_link">
+        <inertial>
+          <origin
+            xyz="0.0 0.0 0.0"
+            rpy="0 0 0" />
+            <mass value="5.71439015182903"/>
+          <inertia
+            ixx="0.00107634033140466"
+            ixy="1.51573650824965E-05"
+            ixz="-6.94838293881106E-05"
+            iyy="0.000914613440717638"
+            iyz="0.000195407309247701"
+            izz="0.000234021785961031" />
+        </inertial>
+      </link>
+    <!-- Add base of wheel macro -->
+    <xacro:asc_wheel wheel_prefix="rear_${wheel_prefix}"
+    link_parent="${link_parent}" wheel_length="${wheel_length}" wheel_radius="${wheel_radius}" >
+    <xacro:insert_block name="wheel_joint_origin"/>
+    <xacro:insert_block name="wheel_joint_axis"/>
+    </xacro:asc_wheel>
+    <!-- Add specfic parts for forward wheels-->
+    <joint name="rear_${wheel_prefix}_steering_joint" type="revolute">
+      <xacro:insert_block name="steering_joint_pose"/>
+      <parent link="${link_parent}"/>
+      <child link="rear_${wheel_prefix}_steering_link"/>
+      <axis xyz="0 0 1"/>
+      <limit
+      lower="0.0"
+      upper="0.0"
+      effort="0"
+      velocity="0" />
     </joint>
   </xacro:macro>

File: sc_description/urdf/macro_link.urdf.xacro (robot description, xacro)
@@ -1,4 +1,4 @@
 <?xml version="1.0"?>
-<robot xmlns:xacro="http://www.ros.org/wiki/xacro" name="asc_link">
+<robot xmlns:xacro="http://ros.org/wiki/xacro" name="asc_link">
 	<xacro:macro name="asc_wheel" params="x_size y_size z_size">
 	<geometry>
