Commit message: removed unnecessary cmakelists

File: asc_description/urdf/asc.urdf.xacro (robot description, xacro)
@@ -110,5 +110,5 @@
   </gazebo>
   <!-- add camera -->
-  <gazebo reference="camera_link">
+  <gazebo reference="zed_camera_center">
     <sensor type="depth" name="openni_camera_camera">
       <always_on>1</always_on>
@@ -172,9 +172,9 @@
      </joint>
   </xacro:if>
-  <link name="camera_link"/>
+  <link name="zed_camera_center"/>
   <joint name="base_to_camera" type="fixed">
-    <origin xyz="1.2 0 0.6" rpy="0 0.1 0"/>
+    <origin xyz="0.142 0 0.54" rpy="0 0 0"/>
     <parent link="base_link"/>
-    <child link="camera_link"/>
+    <child link="zed_camera_center"/>
   </joint>
   <link name="camera_link_pc"/>

Commit message: calibrated camera positioning slightly

File: asc_description/urdf/asc.urdf.xacro (robot description, xacro)
@@ -160,19 +160,29 @@
     <xacro:include filename="$(find velodyne_description)/urdf/VLP-16.urdf.xacro"/>
     <VLP-16 parent="base_link" name="velodyne" topic="/os1_cloud_node/points" hz="10" samples="440" gpu="false">
-      <origin xyz="0.063 0 0.54" rpy="0 0 0"/>
+      <origin xyz="0.063 0 0.53" rpy="0 0 0"/>
     </VLP-16>
   </xacro:if>
   <xacro:if value="${'$(arg simulation)' == 'false'}">
     <!-- Add LiDAR for real -->
-      <link name="os1_sensor"/>
-     <joint name="base_to_os1" type="fixed">
-       <origin xyz="0 0 0" rpy="0 0 0"/>
-       <parent link="base_link"/>
-       <child link="os1_sensor"/>
-     </joint>
+    <link name="os1_sensor"/>
+    <joint name="base_to_os1" type="fixed">
+      <origin xyz="0.063 0 0.53" rpy="0 0 0"/>
+      <parent link="base_link"/>
+      <child link="os1_sensor"/>
+    </joint>
   </xacro:if>
-  <link name="zed_camera_center"/>
+  <link name="zed_camera_center">
+    <visual>
+      <origin xyz="0 0 0" rpy="0 0 0"/>
+      <geometry>
+        <mesh filename="package://zed_wrapper/urdf/models/ZED.stl"/>
+      </geometry>
+      <material name="light_grey">
+        <color rgba="0.8 0.8 0.8 0.8"/>
+      </material>
+    </visual>
+  </link>
   <joint name="base_to_camera" type="fixed">
-    <origin xyz="0.142 0 0.54" rpy="0 0 0"/>
+    <origin xyz="0.149 0 0.49" rpy="0 0 0"/>
     <parent link="base_link"/>
     <child link="zed_camera_center"/>
@@ -181,5 +191,5 @@
   <joint name="camera_to_pc" type="fixed">
     <origin xyz="0 0 0" rpy="-1.57 0 -1.57"/>
-    <parent link="camera_link"/>
+    <parent link="zed_camera_center"/>
     <child link="camera_link_pc"/>
   </joint>

Commit message: added ZED camera mesh to description

File: asc_description/urdf/asc.urdf.xacro (robot description, xacro)
@@ -176,5 +176,5 @@
       <origin xyz="0 0 0" rpy="0 0 0"/>
       <geometry>
-        <mesh filename="package://zed_wrapper/urdf/models/ZED.stl"/>
+        <mesh filename="package://asc_description/meshes/ZED/ZED.stl"/>
       </geometry>
       <material name="light_grey">

Commit message: cleanup of cartographer

File: asc_description/urdf/asc.urdf.xacro (robot description, xacro)
@@ -86,5 +86,5 @@
       <robotNamespace>/</robotNamespace>
       <updateRate>50.0</updateRate>
-      <bodyName>base_link</bodyName>
+      <bodyName>os1_imu</bodyName>
       <topicName>imu/data</topicName>
       <accelDrift>0.005 0.005 0.005</accelDrift>
@@ -157,9 +157,16 @@
   <!-- Add LiDAR -->
   <xacro:if value="${'$(arg simulation)' == 'true'}">
-    <!-- Add LiDAR for simulation-->
+    <!-- Add LiDAR for simulation, pretend it is the os1 LiDAR-->
     <xacro:include filename="$(find velodyne_description)/urdf/VLP-16.urdf.xacro"/>
     <VLP-16 parent="base_link" name="velodyne" topic="/os1_cloud_node/points" hz="10" samples="440" gpu="false">
       <origin xyz="0.063 0 0.53" rpy="0 0 0"/>
     </VLP-16>
+    <!-- connect the os1_sensor to share reference for simulated imu and real imu-->
+    <link name="os1_imu"/>
+        <joint name="base_to_os1" type="fixed">
+      <origin xyz="0 0 0" rpy="0 0 0"/>
+      <parent link="velodyne"/>
+      <child link="os1_imu"/>
+    </joint>
   </xacro:if>
   <xacro:if value="${'$(arg simulation)' == 'false'}">

Commit message: Other settings for interia and mass

File: asc_description/urdf/asc.urdf.xacro (robot description, xacro)
@@ -25,5 +25,5 @@
     <inertial>
       <origin xyz="-0.191135074026536 0.00147037627768998 -0.144166350352701" rpy="0 0 0"/>
-      <mass value="54.6845003989778"/>
+      <mass value="20.0"/>
       <inertia ixx="0.830289508168532" ixy="-7.44170925374484E-07" ixz="-0.168031775231281" iyy="1.89493024064907" iyz="3.6787232173372E-07" izz="1.80540947379668"/>
     </inertial>

File: asc_description/urdf/macro_wheel.urdf.xacro (robot description, xacro)
@@ -5,5 +5,5 @@
       <inertial>
         <origin xyz="-1.02140518265514E-14 6.85007606193722E-14 0.00509989314946457" rpy="0 0 0"/>
-        <mass value="3.6905479088754"/>
+        <mass value="0.3"/>
         <inertia ixx="0.117114266308143" ixy="1.38777878078145E-17" ixz="2.37549730750149E-18" iyy="0.117114266308143" iyz="3.40770700491441E-17" izz="0.22795106404409"/>
       </inertial>
@@ -69,12 +69,12 @@
           xyz="0.0 0.0 0.0"
           rpy="0 0 0" />
-          <mass value="5.71439015182903"/>
+          <mass value="0.5"/>
         <inertia
-          ixx="0.00107634033140466"
-          ixy="1.51573650824965E-05"
-          ixz="-6.94838293881106E-05"
-          iyy="0.000914613440717638"
-          iyz="0.000195407309247701"
-          izz="0.000234021785961031" />
+          ixx="0.138973038944984"
+          ixy="0.00240438901312515"
+          ixz="0.0320681563279578"
+          iyy="0.160053837434921"
+          iyz="-0.0109556260035955"
+          izz="0.028546837728721"/>
       </inertial>
       <visual>
@@ -106,4 +106,5 @@
       <axis xyz="0 0 1"/>
       <limit lower="-0.8" upper="0.9" effort="100" velocity="100"/>
+      <dynamics damping="1.0"/>
     </joint>
   </xacro:macro>
@@ -114,5 +115,5 @@
             xyz="0.0 0.0 0.0"
             rpy="0 0 0" />
-            <mass value="5.71439015182903"/>
+            <mass value="0.3"/>
           <inertia
             ixx="0.00107634033140466"

Commit message: testing of stvl with rolling window seems to work

File: asc_description/urdf/asc.urdf.xacro (robot description, xacro)
@@ -154,4 +154,57 @@
       </plugin>
     </sensor>
+    <sensor type="multicamera" name="stereo_camera">
+      <update_rate>30.0</update_rate>
+      <camera name="left">
+        <horizontal_fov>1.3962634</horizontal_fov>
+        <image>
+          <width>800</width>
+          <height>800</height>
+          <format>R8G8B8</format>
+        </image>
+        <clip>
+          <near>0.02</near>
+          <far>300</far>
+        </clip>
+        <noise>
+          <type>gaussian</type>
+          <mean>0.0</mean>
+          <stddev>0.007</stddev>
+        </noise>
+      </camera>
+      <camera name="right">
+        <pose>0 -0.07 0 0 0 0</pose>
+        <horizontal_fov>1.3962634</horizontal_fov>
+        <image>
+          <width>800</width>
+          <height>800</height>
+          <format>R8G8B8</format>
+        </image>
+        <clip>
+          <near>0.02</near>
+          <far>300</far>
+        </clip>
+        <noise>
+          <type>gaussian</type>
+          <mean>0.0</mean>
+          <stddev>0.007</stddev>
+        </noise>
+      </camera>
+      <plugin name="stereo_camera_controller" filename="libgazebo_ros_multicamera.so">
+        <alwaysOn>true</alwaysOn>
+        <updateRate>0.0</updateRate>
+        <cameraName>multisense_sl/camera</cameraName>
+        <imageTopicName>image_raw</imageTopicName>
+        <cameraInfoTopicName>camera_info</cameraInfoTopicName>
+        <frameName>camera_link_pc</frameName>
+        <!--<rightFrameName>right_camera_optical_frame</rightFrameName>-->
+        <hackBaseline>0.07</hackBaseline>
+        <distortionK1>0.0</distortionK1>
+        <distortionK2>0.0</distortionK2>
+        <distortionK3>0.0</distortionK3>
+        <distortionT1>0.0</distortionT1>
+        <distortionT2>0.0</distortionT2>
+      </plugin>
+    </sensor>
   </gazebo>
   <!-- Add LiDAR -->
@@ -201,46 +254,3 @@
     <child link="camera_link_pc"/>
   </joint>
-  <!--
-  <joint name="zed_camera_center_joint" type="fixed">
-    <parent link="base_link"/>
-    <child link="zed_camera_center"/>
-    <origin xyz="0.16 0 0.07" rpy="0 0 0"/>
-  </joint>
-  <link name="zed_camera_center">
-    <visual>
-      <origin xyz="0 0 0" rpy="0 0 0"/>
-      <geometry>
-        <mesh filename="package://zed_wrapper/urdf/models/ZED.stl"/>
-      </geometry>
-      <material name="light_grey">
-        <color rgba="0.8 0.8 0.8 0.8"/>
-      </material>
-    </visual>
-  </link> -->
-  <!-- Left Camera --> <!--
-  <joint name="zed_left_camera_joint" type="fixed">
-    <parent link="zed_camera_center"/>
-    <child link="zed_left_camera_frame"/>
-    <origin xyz="0 0.06 0" rpy="0 0 0"/>
-  </joint>
-  <link name="zed_left_camera_frame"/>
-  <joint name="zed_left_camera_optical_joint" type="fixed">
-    <origin xyz="0 0 0" rpy="-1.57079632679 0.0 -1.57079632679"/>
-    <parent link="zed_left_camera_frame"/>
-    <child link="zed_left_camera_optical_frame"/>
-  </joint>
-  <link name="zed_left_camera_optical_frame"/> -->
-  <!-- Right Camera --> <!--
-  <joint name="zed_right_camera_joint" type="fixed">
-    <parent link="zed_camera_center"/>
-    <child link="zed_right_camera_frame"/>
-    <origin xyz="0 -0.06 0" rpy="0 0 0"/>
-  </joint>
-  <link name="zed_right_camera_frame"/>
-  <joint name="zed_right_camera_optical_joint" type="fixed">
-    <origin xyz="0 0 0" rpy="-1.57079632679 0.0 -1.57079632679"/>
-    <parent link="zed_right_camera_frame"/>
-    <child link="zed_right_camera_optical_frame"/>
-  </joint>
-  <link name="zed_right_camera_optical_frame"/> -->
 </robot>

Commit message: fixed frames for asc, includes zed

File: asc_description/urdf/asc.urdf.xacro (robot description, xacro)
@@ -254,3 +254,29 @@
     <child link="camera_link_pc"/>
   </joint>
+  <!-- Left Camera -->
+  <joint name="zed_left_camera_joint" type="fixed">
+    <parent link="zed_camera_center"/>
+    <child link="zed_left_camera_frame"/>
+    <origin xyz="0 0.06 0" rpy="0 0 0"/>
+  </joint>
+  <link name="zed_left_camera_frame"/>
+  <joint name="zed_left_camera_optical_joint" type="fixed">
+    <origin xyz="0 0 0" rpy="-1.57079632679 0.0 -1.57079632679"/>
+    <parent link="zed_left_camera_frame"/>
+    <child link="zed_left_camera_optical_frame"/>
+  </joint>
+  <link name="zed_left_camera_optical_frame"/>
+  <!-- Right Camera -->
+  <joint name="zed_right_camera_joint" type="fixed">
+    <parent link="zed_camera_center"/>
+    <child link="zed_right_camera_frame"/>
+    <origin xyz="0 -0.06 0" rpy="0 0 0"/>
+  </joint>
+  <link name="zed_right_camera_frame"/>
+  <joint name="zed_right_camera_optical_joint" type="fixed">
+    <origin xyz="0 0 0" rpy="-1.57079632679 0.0 -1.57079632679"/>
+    <parent link="zed_right_camera_frame"/>
+    <child link="zed_right_camera_optical_frame"/>
+  </joint>
+  <link name="zed_right_camera_optical_frame"/>
 </robot>

Commit message: minor update to parameters

File: asc_description/urdf/asc.urdf.xacro (robot description, xacro)
@@ -244,5 +244,5 @@
   </link>
   <joint name="base_to_camera" type="fixed">
-    <origin xyz="0.149 0 0.49" rpy="0 0 0"/>
+    <origin xyz="0.149 0 0.49" rpy="0 -0.1 0"/> <!-- tune pitch here -->
     <parent link="base_link"/>
     <child link="zed_camera_center"/>

Commit message: fixing missing dependency

File: asc_description/urdf/asc.urdf.xacro (robot description, xacro)
@@ -244,5 +244,5 @@
   </link>
   <joint name="base_to_camera" type="fixed">
-    <origin xyz="0.149 0 0.49" rpy="0 -0.1 0"/> <!-- tune pitch here -->
+    <origin xyz="0.149 0 0.49" rpy="0 -0.1 0"/> <!-- tune pitch here for camera angle-->
     <parent link="base_link"/>
     <child link="zed_camera_center"/>
