Commit message: fixed sc_description to work again

File: sc_description/urdf/sc.urdf.xacro (robot description, xacro)
@@ -24,5 +24,5 @@
       <origin xyz="0 0 0" rpy="0 0 0"/>
       <geometry>
-        <mesh filename="package://asc_description/meshes/base_link.STL"/>
+        <mesh filename="package://sc_description/meshes/base_link.STL"/>
       </geometry>
       <material name="">
@@ -34,5 +34,5 @@
       <origin xyz="0 0 0" rpy="0 0 0"/>
       <geometry>
-        <mesh filename="package://asc_description/meshes/base_link.STL"/>
+        <mesh filename="package://sc_description/meshes/base_link.STL"/>
       </geometry>
     </collision> -->
@@ -47,5 +47,5 @@
       <origin xyz="0 0 0" rpy="0 0 0"/>
       <geometry>
-        <mesh filename="package://asc_description/meshes/left_front_steering_link.STL"/>
+        <mesh filename="package://sc_description/meshes/left_front_steering_link.STL"/>
       </geometry>
       <material name="">
@@ -56,5 +56,5 @@
       <origin xyz="0 0 0" rpy="0 0 0"/>
       <geometry>
-        <mesh filename="package://asc_description/meshes/left_front_steering_link.STL"/>
+        <mesh filename="package://sc_description/meshes/left_front_steering_link.STL"/>
       </geometry>
     </collision>
@@ -101,5 +101,5 @@
       <origin xyz="0 0 0" rpy="0 0 0"/>
       <geometry>
-        <mesh filename="package://asc_description/meshes/right_front_steering_link.STL"/>
+        <mesh filename="package://sc_description/meshes/right_front_steering_link.STL"/>
       </geometry>
       <material name="">
@@ -110,5 +110,5 @@
       <origin xyz="0 0 0" rpy="0 0 0"/>
       <geometry>
-        <mesh filename="package://asc_description/meshes/right_front_steering_link.STL"/>
+        <mesh filename="package://sc_description/meshes/right_front_steering_link.STL"/>
       </geometry>
     </collision>
